Commit message: gazebo test without gripper

File: cora_gripper_1_description/urdf/cora_gripper.ros2_control.xacro (robot description, xacro)
@@ -14,11 +14,19 @@
                 <param name="can">can0</param>
               </xacro:if>
+              <!-- Gazebo hardware components -->
+              <xacro:if value="${hardware_type == 'Gazebo'}">
+                <plugin>gz_ros2_control/GazeboSimSystem</plugin>
+              </xacro:if>
             </hardware>
             <joint name="Finger1">
                 <command_interface name="position"/>
-                <command_interface name="velocity"/>
+                <!-- <command_interface name="velocity"/> -->
                 <state_interface name="position">
                   <param name="initial_value">${initial_positions['Finger1']}</param>
                 </state_interface>
+                <state_interface name="velocity"/>
+                <param name="node_id">6</param>
+            </joint>
+            <joint name="Finger2">
                 <state_interface name="position"/>
                 <state_interface name="velocity"/>

File: cora_moveit_config/config/cora.urdf.xacro (robot description, xacro)
@@ -39,13 +39,5 @@
             initial_positions_file="$(arg initial_positions_file)"/>
     </xacro:if>
-    <!-- ===================== -->
-    <!--     Gazebo plugin     -->
-    <!-- ===================== -->
-    </xacro:if value="${hardware_type == 'Gazebo'}">
-        <gazebo>
-            <plugin filename="libgz_ros2_control-system.so" name="gz_ros2_control::GazeboSimROS2ControlPlugin">
-                <parameters>$(find cora_moveit_config)/config/ros2_controllers.yaml</parameters>
-            </plugin>
-        </gazebo>
-    </xacro:if>
+    <xacro:include filename="$(find cora_gazebo)/config/cora_gazebo.xacro"/>
+    <xacro:cora_gazebo/>
 </robot>
