Commit message: added todo's and issues

File: cora_gripper_1_description/urdf/cora_gripper.ros2_control.xacro (robot description, xacro)
@@ -1,3 +1,11 @@
 <?xml version="1.0"?>
+<!-- TODO: #3 Collapse these two copy-pasted <joint> blocks into ONE recursive
+     xacro macro driven by the generated robot_layout.yaml. The node_id values
+     (6) are hardcoded here but are only known to the configurator.
+     This file already loads YAML for initial_positions — extend that to the
+     joint list itself. Verified working on Jazzy; pattern and gotchas
+     (&lt; escaping, no set() in the sandbox) are in C-O-R-A/cora_common#3. -->
+<!-- TODO: #3 Finger2 is a state-only mimic joint (no command_interface).
+     robot_layout.yaml needs a mimic_joints map to express this. -->
 <robot xmlns:xacro="http://www.ros.org/wiki/xacro">
     <xacro:macro name="cora_gripper_ros2_control" params="name initial_positions_file hardware_type">

File: cora_moveit_config/config/cora.ros2_control.xacro (robot description, xacro)
@@ -1,3 +1,9 @@
 <?xml version="1.0"?>
+<!-- TODO: #3 Collapse these six copy-pasted <joint> blocks into ONE recursive
+     xacro macro driven by the generated robot_layout.yaml. The node_id values
+     (0-5) are hardcoded here but are only known to the configurator.
+     This file already loads YAML for initial_positions — extend that to the
+     joint list itself. Verified working on Jazzy; pattern and gotchas
+     (&lt; escaping, no set() in the sandbox) are in C-O-R-A/cora_common#3. -->
 <robot xmlns:xacro="http://www.ros.org/wiki/xacro">
     <xacro:macro name="cora_ros2_control" params="name initial_positions_file hardware_type">

File: cora_moveit_config/config/cora.urdf.xacro (robot description, xacro)
@@ -1,3 +1,12 @@
 <?xml version="1.0"?>
+<!-- TODO: #3 GENERATED ARTIFACT — the configurator must emit this top-level file,
+     not just the bare kinematic chain it produces today. Missing from its output:
+     the hardware_type/gripper_package/initial_positions_file args, the ros2_control
+     include, and the Gazebo branch. See C-O-R-A/configurator#4.
+     NOTE: this file must stay GENERATED TEXT, not a generic file that loops
+     robot_layout.yaml — xacro:include with a computed filename inside a macro does
+     not register the included macros, and the joint-library macros take *origin as
+     a block param that cannot be built from YAML. Verified on Jazzy; see
+     C-O-R-A/configurator#1. -->
 <robot xmlns:xacro="http://www.ros.org/wiki/xacro" name="cora">
     <!-- ================= -->

File: cora_moveit_config/config/cora_gazebo.ros2_control.xacro (robot description, xacro)
@@ -1,3 +1,9 @@
 <?xml version="1.0"?>
+<!-- TODO: #3 Collapse these six copy-pasted <joint> blocks into ONE recursive
+     xacro macro driven by the generated robot_layout.yaml. The node_id values
+     (none here, but the joint list is still unrolled) are hardcoded here but are only known to the configurator.
+     This file already loads YAML for initial_positions — extend that to the
+     joint list itself. Verified working on Jazzy; pattern and gotchas
+     (&lt; escaping, no set() in the sandbox) are in C-O-R-A/cora_common#3. -->
 <robot xmlns:xacro="http://www.ros.org/wiki/xacro">
     <xacro:macro name="cora_gazebo_ros2_control" params="initial_positions_file">
