Commit message: update urdf file paths

File: cora_description/urdf/cora.urdf (robot description, URDF)
Before this commit: robot cora, 8 links, 7 joints
Links:
- link baselink: geometry collision mesh filename=file://$(find cora_description)/meshes/cora/merged/baselink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; visual mesh filename=file://$(find cora_description)/meshes/cora/merged/baselink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
- link endeffector: geometry collision mesh filename=file://$(find cora_description)/meshes/cora/merged/endeffec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; visual mesh filename=file://$(find cora_description)/meshes/cora/merged/endeffec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
- link l1: geometry collision mesh filename=file://$(find cora_description)/meshes/cora/merged/l1_colli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; visual mesh filename=file://$(find cora_description)/meshes/cora/merged/l1_visua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
- link l2: geometry collision mesh filename=file://$(find cora_description)/meshes/cora/merged/l2_colli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; visual mesh filename=file://$(find cora_description)/meshes/cora/merged/l2_visua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
- link l3: geometry collision mesh filename=file://$(find cora_description)/meshes/cora/merged/l3_colli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; visual mesh filename=file://$(find cora_description)/meshes/cora/merged/l3_visua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
- link l4: geometry collision mesh filename=file://$(find cora_description)/meshes/cora/merged/l4_colli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; visual mesh filename=file://$(find cora_description)/meshes/cora/merged/l4_visua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
- link l5: geometry collision mesh filename=file://$(find cora_description)/meshes/cora/merged/l5_colli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; visual mesh filename=file://$(find cora_description)/meshes/cora/merged/l5_visua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

Commit message: gazebo segfaults for no reason. no idea how to fix

File: cora_description/urdf/cora.urdf (robot description, URDF)
Before this commit: robot cora, 8 links, 7 joints
Links:
- link base_link: mass 1e-09 -> None

File: cora_moveit_config/config/cora.urdf.xacro (robot description, xacro)
@@ -14,9 +14,24 @@
     <!-- ros2_control      -->
     <!-- ================= -->
-    <xacro:include filename="cora.ros2_control.xacro"/>
-    <xacro:cora_ros2_control
-        name="CoraSystem"
-        hardware_type="$(arg hardware_type)"
-        initial_positions_file="$(arg initial_positions_file)"/>
+    <!-- Store hardware_type -->
+    <xacro:property
+        name="hardware_type"
+        value="$(arg hardware_type)"/>
+    <xacro:if value="${hardware_type != 'Gazebo'}">
+        <xacro:include filename="cora.ros2_control.xacro"/>
+        <xacro:cora_ros2_control
+            name="CoraSystem"
+            hardware_type="$(arg hardware_type)"
+            initial_positions_file="$(arg initial_positions_file)"/>
+    </xacro:if>
+    <xacro:if value="${hardware_type == 'Gazebo'}">
+        <!-- gazebo ros2 control configuration -->
+        <xacro:include filename="cora_gazebo.ros2_control.xacro"/>
+        <xacro:cora_gazebo_ros2_control
+            initial_positions_file="$(arg initial_positions_file)"/>
+        <!-- gazebo sensors and plugins -->
+        <xacro:include filename="$(find cora_gazebo)/config/cora_gazebo.xacro"/>
+        <xacro:cora_gazebo/>
+    </xacro:if>
     <!-- ================= -->
     <!-- Optional gripper  -->
@@ -39,5 +54,3 @@
             initial_positions_file="$(arg initial_positions_file)"/>
     </xacro:if>
-    <xacro:include filename="$(find cora_gazebo)/config/cora_gazebo.xacro"/>
-    <xacro:cora_gazebo/>
 </robot>

Commit message: new collision meshes

File: cora_description/urdf/cora.urdf (robot description, URDF)
Before this commit: robot cora, 8 links, 7 joints
Links:
- link base_link: mass None -> 0
- link baselink: geometry collision mesh filename=file://$(find cora_description)/meshes/baselink_collision.s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; visual mesh filename=file://$(find cora_description)/meshes/baselink_visual.dae
- link endeffector: mass 1e-09 -> 0.05; geometry collision mesh filename=file://$(find cora_description)/meshes/endeffector_collisio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; visual mesh filename=file://$(find cora_description)/meshes/endeffector_visual.d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
- link l1: geometry collision mesh filename=file://$(find cora_description)/meshes/l1_collision.stl; visual mesh filename=file://$(find cora_description)/meshes/l1_visual.dae
- link l2: geometry collision mesh filename=file://$(find cora_description)/meshes/l2_collision.stl; visual mesh filename=file://$(find cora_description)/meshes/l2_visual.dae
- link l3: geometry collision mesh filename=file://$(find cora_description)/meshes/l3_collision.stl; visual mesh filename=file://$(find cora_description)/meshes/l3_visual.dae
- link l4: geometry collision mesh filename=file://$(find cora_description)/meshes/l4_collision.stl; visual mesh filename=file://$(find cora_description)/meshes/l4_visual.dae
- link l5: geometry collision mesh filename=file://$(find cora_description)/meshes/l5_collision.stl; visual mesh filename=file://$(find cora_description)/meshes/l5_visual.dae
Joints:
- joint J1: origin xyz=1.08655e-17 -5.35667e-26 0.139 rpy=-3.14159 -1.07316e-15 0.523599 -> xyz=0 0 0.139 rpy=-3.14159 0 0.523599
- joint J2: origin xyz=0.0900666 0.052 -0.088 rpy=-1.5708 1.0472 2.0944 -> xyz=0.090067 0.052 -0.088 rpy=1.570793 2.094393 -1.047192
- joint J3: origin xyz=0.393176 0.227 0.002 rpy=-3.14159 -1.73694e-15 -1.0472 -> xyz=0.393176 0.227 0.002 rpy=-3.14159 0 -1.0472
- joint J4: origin xyz=-2.23477e-15 -0.335 -0.0138333 rpy=-3.14159 -5.25775e-15 -1.77358e-14 -> xyz=0 -0.335 -0.013833 rpy=-3.14159 0 0
- joint J5: origin xyz=4.46411e-16 0.0811667 -0.075 rpy=1.5708 -6.65049e-14 -4.10783e-15 -> xyz=0 0.081167 -0.075 rpy=1.5708 0 0
- joint J6: origin xyz=-1.79316e-15 0.0801667 -0.075 rpy=1.5708 -1.5708 0 -> xyz=0 0.080167 -0.075 rpy=1.5708 -1.570793 0
- joint base_link_to_baselink: axis 0 0 1 -> (none); limit effort=10 velocity=10 -> (none); origin xyz=0 0 0 rpy=0 -0 0 -> (none)
